File: pcb/go-kart-esc/DRV8701P-A.kicad_sch (KiCad schematic)
At the start: 3 parts

Commit message: Poggers
Parts:
- added C5, C6, C7: 1u, symbol Device:C_Small
- added C8: 10u, symbol Device:C_Small
- added R2 (x2): 10k, symbol Device:R
Connections:
- net +3V3: now also C5.1
- net +4V: now also C6.1, R2.1
- net GND: now also U1.20 (SN), U1.21 (SP), U1.6 (VREF), C5.2, C6.2, C7.2, C8.2, R2.2
- net IDRIVE: now reaches U1.12 (IDRIVE)
- net IDRIVE: now also R2.1, R2.2
- new net: C7.1, C8.1

Commit message: ooga booga
Parts:
- C201: renamed from C1; footprint (none) -> Capacitor_SMD:C_0603_1608Metric_Pad1.08x0.95mm_HandSolder
- C202: renamed from C2; footprint (none) -> Capacitor_SMD:C_0603_1608Metric_Pad1.08x0.95mm_HandSolder
- C203: renamed from C5; footprint (none) -> Capacitor_SMD:C_0603_1608Metric_Pad1.08x0.95mm_HandSolder
- C204: renamed from C6; footprint (none) -> Capacitor_SMD:C_0603_1608Metric_Pad1.08x0.95mm_HandSolder
- C205: renamed from C7; footprint (none) -> Capacitor_SMD:C_0603_1608Metric_Pad1.08x0.95mm_HandSolder
- C206: renamed from C8; footprint (none) -> Capacitor_SMD:C_0805_2012Metric_Pad1.18x1.45mm_HandSolder
- R2: footprint (none) -> Resistor_SMD:R_0402_1005Metric_Pad0.72x0.64mm_HandSolder
- U201: renamed from U1; value ~ -> DRV8701PRGER; footprint (none) -> Package_DFN_QFN:Texas_S-PVQFN-N24_EP2.1x2.1mm
Connections:
- net +BATT: now reaches U201.1 (VM)
- net +BATT: now also C205.1, C206.1

Commit message: ooga booga
Parts:
- C202: value 1u -> 0.1u; footprint Capacitor_SMD:C_0603_1608Metric_Pad1.08x0.95mm_HandSolder -> Capacitor_SMD:C_0402_1005Metric_Pad0.74x0.62mm_HandSolder
Connections:
- net +BATT: now also C201.1
- net GND: now also U201.25 (GND); no longer U201.PPAD (GND)
Other:
- moved on the sheet: U201
Changed lines of the file:
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@@
     (pin "8")
     (pin "9")
-    (pin "PPAD")
+    (pin "25")
     (instances
       (project "go-kart-esc"
@@
         )
         (path "/5a70b585-4866-4f79-8013-f2242aeded57/2a07445c-1516-44d0-a079-c83f7310c200"
-          (reference "#PWR0209") (unit 1)
-        )
-        (path "/5a70b585-4866-4f79-8013-f2242aeded57/273f23de-e221-4afe-873d-53a6030e7e3a"
-          (reference "#PWR0509") (unit 1)
+          (reference "#PWR0213") (unit 1)
+        )
+        (path "/5a70b585-4866-4f79-8013-f2242aeded57/273f23de-e221-4afe-873d-53a6030e7e3a"
+          (reference "#PWR0513") (unit 1)
         )
       )
@@
     )
   )
+  (symbol (lib_id "power:+BATT") (at 157.48 64.77 0) (unit 1)
+    (in_bom yes) (on_board yes) (dnp no) (fields_autoplaced)
+    (property "Reference" "#PWR0601" (at 157.48 68.58 0)
+      (effects (font (size 1.27 1.27)) hide)
+    )
+    (property "Value" "+BATT" (at 157.48 59.69 0)
+      (effects (font (size 1.27 1.27)))
+    )
+    (property "Footprint" "" (at 157.48 64.77 0)
+      (effects (font (size 1.27 1.27)) hide)
+    )
+    (property "Datasheet" "" (at 157.48 64.77 0)
+      (effects (font (size 1.27 1.27)) hide)
+    )
+    (pin "1")
+    (instances
+      (project "go-kart-esc"
+        (path "/5a70b585-4866-4f79-8013-f2242aeded57/a459c41b-c6c3-40c7-8485-5a95e06155ac"
+          (reference "#PWR0601") (unit 1)
+        )
+        (path "/5a70b585-4866-4f79-8013-f2242aeded57/2f2eb473-a6d5-4b09-8c58-ce0c11f580af"
+          (reference "#PWR0301") (unit 1)
+        )
+        (path "/5a70b585-4866-4f79-8013-f2242aeded57/2a07445c-1516-44d0-a079-c83f7310c200"
+          (reference "#PWR0209") (unit 1)
+        )
+        (path "/5a70b585-4866-4f79-8013-f2242aeded57/273f23de-e221-4afe-873d-53a6030e7e3a"
+          (reference "#PWR0509") (unit 1)
+        )
+      )
+    )
+  )
   (symbol (lib_id "power:GND") (at 226.06 71.12 0) (unit 1)
     (in_bom yes) (on_board yes) (dnp no) (fields_autoplaced)
@@
       (effects (font (size 1.27 1.27)) (justify left))
     )
-    (property "Value" "1u" (at 168.91 80.0163 0)
-      (effects (font (size 1.27 1.27)) (justify left))
-    )
-    (property "Footprint" "Capacitor_SMD:C_0603_1608Metric_Pad1.08x0.95mm_HandSolder" (at 166.37 78.74 0)
+    (property "Value" "0.1u" (at 168.91 80.0163 0)
+      (effects (font (size 1.27 1.27)) (justify left))
+    )
+    (property "Footprint" "Capacitor_SMD:C_0402_1005Metric_Pad0.74x0.62mm_HandSolder" (at 166.37 78.74 0)
       (effects (font (size 1.27 1.27)) hide)
     )
@@
         )
       )
-    )
-  )
-  (symbol (lib_id "ESC:VM") (at 157.48 64.77 0) (unit 1)
-    (in_bom no) (on_board no) (dnp no) (fields_autoplaced)
-    (property "Reference" "#PWR0126" (at 152.4 62.23 0)
-      (effects (font (size 1.27 1.27)) hide)
-    )
-    (property "Value" "VM" (at 157.48 59.69 0)
-      (effects (font (size 1.27 1.27)))
-    )
-    (property "Footprint" "" (at 157.48 64.77 0)
-      (effects (font (size 1.27 1.27)) hide)
-    )
-    (property "Datasheet" "" (at 157.48 64.77 0)
-      (effects (font (size 1.27 1.27)) hide)
-    )
-    (pin "1")
-    (instances
-      (project "go-kart-esc"
-        (path "/5a70b585-4866-4f79-8013-f2242aeded57/2a07445c-1516-44d0-a079-c83f7310c200"
-          (reference "#PWR0126") (unit 1)
-        )
-        (path "/5a70b585-4866-4f79-8013-f2242aeded57/273f23de-e221-4afe-873d-53a6030e7e3a"
-          (reference "#PWR0131") (unit 1)
-        )
-      )

Commit message: Began Routing
Parts:
- removed C206: 10u, Capacitor_SMD:C_0805_2012Metric_Pad1.18x1.45mm_HandSolder, symbol Device:C_Small
- removed R2 (x2): 10k, Resistor_SMD:R_0402_1005Metric_Pad0.72x0.64mm_HandSolder, symbol Device:R
- added C206: 10u@50V, Capacitor_SMD:CP_Elec_5x5.8, symbol Device:C_Polarized_Small
- C201, C203, C204: footprint Capacitor_SMD:C_0603_1608Metric_Pad1.08x0.95mm_HandSolder -> Capacitor_SMD:C_0402_1005Metric_Pad0.74x0.62mm_HandSolder
- C202: value 0.1u -> 0.1u@50V; footprint Capacitor_SMD:C_0402_1005Metric_Pad0.74x0.62mm_HandSolder -> Capacitor_SMD:C_0603_1608Metric_Pad1.08x0.95mm_HandSolder
- C205: value 1u -> 1u@50V; footprint Capacitor_SMD:C_0603_1608Metric_Pad1.08x0.95mm_HandSolder -> Capacitor_SMD:C_0402_1005Metric_Pad0.74x0.62mm_HandSolder
Connections:
- net IDRIVE is gone; now on net GND: U201.12 (IDRIVE)
- net +BATT: now also C206.1
- net GND: now also C206.2

Commit message: Theory can only take you so far.
Connections:
- net +3V3: no longer names the net of C203.1, U201.8 (DVDD)
- net +4V: no longer names the net of C204.1, U201.7 (AVDD)
Changed lines of the file:
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@@
     (stroke (width 0) (type default))
   )
-  (wire (pts (xy 139.7 64.77) (xy 139.7 67.31))
+  (wire (pts (xy 139.7 44.45) (xy 139.7 67.31))
     (stroke (width 0) (type default))
   )
@@
     (stroke (width 0) (type default))
   )
+  (wire (pts (xy 137.16 57.15) (xy 194.31 57.15))
+    (stroke (width 0) (type default))
+  )
   (wire (pts (xy 87.63 115.57) (xy 96.52 115.57))
     (stroke (width 0) (type default))
@@
     (stroke (width 0) (type default))
   )
-  (wire (pts (xy 137.16 60.96) (xy 137.16 67.31))
+  (wire (pts (xy 137.16 57.15) (xy 137.16 67.31))
     (stroke (width 0) (type default))
   )
@@
     (stroke (width 0) (type default))
   )
+  (wire (pts (xy 205.74 44.45) (xy 205.74 60.96))
+    (stroke (width 0) (type default))
+  )
   (wire (pts (xy 87.63 115.57) (xy 87.63 130.81))
     (stroke (width 0) (type default))
@@
     (stroke (width 0) (type default))
   )
+  (wire (pts (xy 139.7 44.45) (xy 205.74 44.45))
+    (stroke (width 0) (type default))
+  )
   (wire (pts (xy 156.21 105.41) (xy 156.21 109.22))
     (stroke (width 0) (type default))
@@
   )
   (wire (pts (xy 194.31 66.04) (xy 194.31 67.31))
-    (stroke (width 0) (type default))
-  )
-  (wire (pts (xy 205.74 57.15) (xy 205.74 60.96))
     (stroke (width 0) (type default))
   )
@@
     )
   )
-  (symbol (lib_id "power:+4V") (at 205.74 57.15 0) (unit 1)
-    (in_bom yes) (on_board yes) (dnp no) (fields_autoplaced)
-    (property "Reference" "#PWR0212" (at 205.74 60.96 0)
-      (effects (font (size 1.27 1.27)) hide)
-    )
-    (property "Value" "+4V" (at 205.74 52.07 0)
-      (effects (font (size 1.27 1.27)))
-    )
-    (property "Footprint" "" (at 205.74 57.15 0)
-      (effects (font (size 1.27 1.27)) hide)
-    )
-    (property "Datasheet" "" (at 205.74 57.15 0)
-      (effects (font (size 1.27 1.27)) hide)
-    )
-    (pin "1")
-    (instances
-      (project "go-kart-esc"
-        (path "/5a70b585-4866-4f79-8013-f2242aeded57/2a07445c-1516-44d0-a079-c83f7310c200"
-          (reference "#PWR0212") (unit 1)
-        )
-        (path "/5a70b585-4866-4f79-8013-f2242aeded57/273f23de-e221-4afe-873d-53a6030e7e3a"
-          (reference "#PWR0512") (unit 1)
-        )
-      )
-    )
-  )
   (symbol (lib_id "Device:C_Small") (at 157.48 71.12 0) (unit 1)
     (in_bom yes) (on_board yes) (dnp no) (fields_autoplaced)
@@
         (path "/5a70b585-4866-4f79-8013-f2242aeded57/273f23de-e221-4afe-873d-53a6030e7e3a"
           (reference "C501") (unit 1)
-        )
-      )
-    )
-  )
-  (symbol (lib_id "power:+3V3") (at 194.31 57.15 0) (unit 1)
-    (in_bom yes) (on_board yes) (dnp no) (fields_autoplaced)
-    (property "Reference" "#PWR0210" (at 194.31 60.96 0)
-      (effects (font (size 1.27 1.27)) hide)
-    )
-    (property "Value" "+3V3" (at 194.31 52.07 0)
-      (effects (font (size 1.27 1.27)))
-    )
-    (property "Footprint" "" (at 194.31 57.15 0)
-      (effects (font (size 1.27 1.27)) hide)
-    )
-    (property "Datasheet" "" (at 194.31 57.15 0)
-      (effects (font (size 1.27 1.27)) hide)
-    )
-    (pin "1")
-    (instances
-      (project "go-kart-esc"
-        (path "/5a70b585-4866-4f79-8013-f2242aeded57/2a07445c-1516-44d0-a079-c83f7310c200"
-          (reference "#PWR0210") (unit 1)
-        )
-        (path "/5a70b585-4866-4f79-8013-f2242aeded57/273f23de-e221-4afe-873d-53a6030e7e3a"
-          (reference "#PWR0510") (unit 1)
         )
       )
@@
     )
   )
-  (symbol (lib_id "power:+3V3") (at 137.16 60.96 0) (unit 1)
-    (in_bom yes) (on_board yes) (dnp no) (fields_autoplaced)
-    (property "Reference" "#PWR0204" (at 137.16 64.77 0)
-      (effects (font (size 1.27 1.27)) hide)
-    )
-    (property "Value" "+3V3" (at 137.16 55.88 0)
-      (effects (font (size 1.27 1.27)))
-    )
-    (property "Footprint" "" (at 137.16 60.96 0)
-      (effects (font (size 1.27 1.27)) hide)
-    )
-    (property "Datasheet" "" (at 137.16 60.96 0)
-      (effects (font (size 1.27 1.27)) hide)
-    )
-    (pin "1")
-    (instances
-      (project "go-kart-esc"
-        (path "/5a70b585-4866-4f79-8013-f2242aeded57/2a07445c-1516-44d0-a079-c83f7310c200"
-          (reference "#PWR0204") (unit 1)
-        )
-        (path "/5a70b585-4866-4f79-8013-f2242aeded57/273f23de-e221-4afe-873d-53a6030e7e3a"
-          (reference "#PWR0504") (unit 1)
-        )
-      )
-    )
-  )
   (symbol (lib_id "Device:C_Small") (at 205.74 63.5 0) (unit 1)
     (in_bom yes) (on_board yes) (dnp no) (fields_autoplaced)
@@
         )
       )
-    )
-  )
-  (symbol (lib_id "power:+4V") (at 139.7 64.77 0) (unit 1)
-    (in_bom yes) (on_board yes) (dnp no) (fields_autoplaced)
-    (property "Reference" "#PWR0205" (at 139.7 68.58 0)
-      (effects (font (size 1.27 1.27)) hide)
-    )
-    (property "Value" "+4V" (at 139.7 59.69 0)
-      (effects (font (size 1.27 1.27)))
-    )
-    (property "Footprint" "" (at 139.7 64.77 0)
-      (effects (font (size 1.27 1.27)) hide)
-    )
-    (property "Datasheet" "" (at 139.7 64.77 0)
-      (effects (font (size 1.27 1.27)) hide)
-    )
-    (pin "1")
-    (instances
-      (project "go-kart-esc"
-        (path "/5a70b585-4866-4f79-8013-f2242aeded57/2a07445c-1516-44d0-a079-c83f7310c200"
-          (reference "#PWR0205") (unit 1)
-        )
-        (path "/5a70b585-4866-4f79-8013-f2242aeded57/273f23de-e221-4afe-873d-53a6030e7e3a"
-          (reference "#PWR0505") (unit 1)
-        )
-      )

Commit message: Finished PCB
Parts:
- renumbered C201 to C501, C202 to C502, C203 to C503, C204 to C504, C205 to C505, C206 to C506, U201 to U501
