File: pcb/go-kart-esc/STM32F042.kicad_sch (KiCad schematic)
At the start: 9 parts, among them U3 STM32F042C6Ux

Commit message: ooga booga
Parts:
- C3: footprint (none) -> Capacitor_SMD:C_0603_1608Metric_Pad1.08x0.95mm_HandSolder
- C3: footprint (none) -> Capacitor_SMD:C_0402_1005Metric_Pad0.74x0.62mm_HandSolder
- renumbered U3 to U401
Changed lines of the file:
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@@
       (effects (font (size 1.27 1.27)) (justify left))
     )
-    (property "Footprint" "" (at 242.2652 54.61 0)
+    (property "Footprint" "Capacitor_SMD:C_0603_1608Metric_Pad1.08x0.95mm_HandSolder" (at 242.2652 54.61 0)
       (effects (font (size 1.27 1.27)) hide)
     )
@@
         )
         (path "/5a70b585-4866-4f79-8013-f2242aeded57/2a126528-6fa8-4cd4-ac38-dfc3256831d3"
-          (reference "C15") (unit 1)
+          (reference "C406") (unit 1)
         )
       )
@@
         )
         (path "/5a70b585-4866-4f79-8013-f2242aeded57/2a126528-6fa8-4cd4-ac38-dfc3256831d3"
-          (reference "#PWR030") (unit 1)
+          (reference "#PWR0402") (unit 1)
         )
       )
@@
       (effects (font (size 1.27 1.27)) (justify left))
     )
-    (property "Footprint" "" (at 216.8652 54.61 0)
+    (property "Footprint" "Capacitor_SMD:C_0402_1005Metric_Pad0.74x0.62mm_HandSolder" (at 216.8652 54.61 0)
       (effects (font (size 1.27 1.27)) hide)
     )
@@
         )
         (path "/5a70b585-4866-4f79-8013-f2242aeded57/2a126528-6fa8-4cd4-ac38-dfc3256831d3"
-          (reference "C13") (unit 1)
+          (reference "C404") (unit 1)
         )
       )
@@
   (symbol (lib_id "MCU_ST_STM32F0:STM32F042C6Ux") (at 148.59 114.3 0) (unit 1)
     (in_bom yes) (on_board yes) (dnp no) (fields_autoplaced)
-    (property "Reference" "U3" (at 153.3241 152.4 0)
+    (property "Reference" "U401" (at 153.3241 152.4 0)
       (effects (font (size 1.27 1.27)) (justify left))
     )
@@
       (project "go-kart-esc"
         (path "/5a70b585-4866-4f79-8013-f2242aeded57/2a126528-6fa8-4cd4-ac38-dfc3256831d3"
-          (reference "U3") (unit 1)
+          (reference "U401") (unit 1)
         )
       )
@@
         )
         (path "/5a70b585-4866-4f79-8013-f2242aeded57/2a126528-6fa8-4cd4-ac38-dfc3256831d3"
-          (reference "#PWR032") (unit 1)
+          (reference "#PWR0405") (unit 1)
         )
       )
@@
         )
         (path "/5a70b585-4866-4f79-8013-f2242aeded57/2a126528-6fa8-4cd4-ac38-dfc3256831d3"
-          (reference "#PWR031") (unit 1)
+          (reference "#PWR0404") (unit 1)
         )
       )
@@
       (effects (font (size 1.27 1.27)) (justify left))
     )
-    (property "Footprint" "" (at 190.1952 54.61 0)
+    (property "Footprint" "Capacitor_SMD:C_0402_1005Metric_Pad0.74x0.62mm_HandSolder" (at 190.1952 54.61 0)
       (effects (font (size 1.27 1.27)) hide)
     )
@@
         )
         (path "/5a70b585-4866-4f79-8013-f2242aeded57/2a126528-6fa8-4cd4-ac38-dfc3256831d3"
-          (reference "C11") (unit 1)
+          (reference "C402") (unit 1)
         )
       )
@@
       (effects (font (size 1.27 1.27)) (justify left))
     )
-    (property "Footprint" "" (at 120.3452 91.44 0)
+    (property "Footprint" "Capacitor_SMD:C_0402_1005Metric_Pad0.74x0.62mm_HandSolder" (at 120.3452 91.44 0)
       (effects (font (size 1.27 1.27)) hide)
     )
@@
         )
         (path "/5a70b585-4866-4f79-8013-f2242aeded57/2a126528-6fa8-4cd4-ac38-dfc3256831d3"
-          (reference "C18") (unit 1)
+          (reference "C401") (unit 1)
         )
       )
@@
         )
         (path "/5a70b585-4866-4f79-8013-f2242aeded57/2a126528-6fa8-4cd4-ac38-dfc3256831d3"
-          (reference "#PWR029") (unit 1)
+          (reference "#PWR0403") (unit 1)
         )
       )
@@
       (effects (font (size 1.27 1.27)) (justify left))
     )
-    (property "Footprint" "" (at 229.5652 54.61 0)
+    (property "Footprint" "Capacitor_SMD:C_0603_1608Metric_Pad1.08x0.95mm_HandSolder" (at 229.5652 54.61 0)
       (effects (font (size 1.27 1.27)) hide)
     )
@@
         )
         (path "/5a70b585-4866-4f79-8013-f2242aeded57/2a126528-6fa8-4cd4-ac38-dfc3256831d3"
-          (reference "C14") (unit 1)
+          (reference "C405") (unit 1)
         )
       )
@@
         )
         (path "/5a70b585-4866-4f79-8013-f2242aeded57/2a126528-6fa8-4cd4-ac38-dfc3256831d3"
-          (reference "#PWR033") (unit 1)
+          (reference "#PWR0401") (unit 1)
         )
       )
@@
       (effects (font (size 1.27 1.27)) (justify left))
     )
-    (property "Footprint" "" (at 267.6652 54.61 0)
+    (property "Footprint" "Capacitor_SMD:C_0603_1608Metric_Pad1.08x0.95mm_HandSolder" (at 267.6652 54.61 0)
       (effects (font (size 1.27 1.27)) hide)
     )
@@
         )
         (path "/5a70b585-4866-4f79-8013-f2242aeded57/2a126528-6fa8-4cd4-ac38-dfc3256831d3"
-          (reference "C17") (unit 1)
+          (reference "C408") (unit 1)
         )
       )
@@
       (effects (font (size 1.27 1.27)) (justify left))
     )
-    (property "Footprint" "" (at 204.1652 54.61 0)
+    (property "Footprint" "Capacitor_SMD:C_0402_1005Metric_Pad0.74x0.62mm_HandSolder" (at 204.1652 54.61 0)
       (effects (font (size 1.27 1.27)) hide)
     )
@@
         )
         (path "/5a70b585-4866-4f79-8013-f2242aeded57/2a126528-6fa8-4cd4-ac38-dfc3256831d3"
-          (reference "C12") (unit 1)
+          (reference "C403") (unit 1)
         )
       )
@@
       (effects (font (size 1.27 1.27)) (justify left))
     )
-    (property "Footprint" "" (at 254.9652 54.61 0)
+    (property "Footprint" "Capacitor_SMD:C_0402_1005Metric_Pad0.74x0.62mm_HandSolder" (at 254.9652 54.61 0)
       (effects (font (size 1.27 1.27)) hide)
     )
@@
         )
         (path "/5a70b585-4866-4f79-8013-f2242aeded57/2a126528-6fa8-4cd4-ac38-dfc3256831d3"
-          (reference "C16") (unit 1)
-        )
-      )
+          (reference "C407") (unit 1)
+        )
+      )

Commit message: Began Routing
Parts:
- C3: footprint Capacitor_SMD:C_0603_1608Metric_Pad1.08x0.95mm_HandSolder -> Capacitor_SMD:C_0402_1005Metric_Pad0.74x0.62mm_HandSolder
Connections:
- net +3V3: now also C3.1, C3.1, C3.1, C3.1, C3.1, C3.1, C3.1
- net PHASE1_A: now also U401.30 (PA9); no longer U401.31 (PA10)
- net PHASE1_B: now also U401.32 (PA11); no longer U401.29 (PA8)
- net PHASE2_A: now also U401.29 (PA8); no longer U401.32 (PA11)
- net PHASE2_B: now also U401.31 (PA10); no longer U401.30 (PA9)
- net nFAULT_A: now also U401.25 (PB12); no longer U401.27 (PB14)
- net nFAULT_B: now also U401.27 (PB14); no longer U401.25 (PB12)
- net nSLEEP_A: now also U401.26 (PB13); no longer U401.28 (PB15)
- net nSLEEP_B: now also U401.28 (PB15); no longer U401.26 (PB13)

Commit message: Finished PCB
Parts:
- renumbered C3 to C401, C3 to C402, C3 to C403, C3 to C404, C3 to C405, C3 to C406, C3 to C407, C3 to C408
