File: pcb/go-kart-esc/can.kicad_sch (KiCad schematic)
At the start: 4 parts

Commit message: ooga booga
Parts:
- C3: footprint (none) -> Capacitor_SMD:C_0402_1005Metric_Pad0.74x0.62mm_HandSolder
- R4: value 220 -> 120; footprint (none) -> Resistor_SMD:R_0402_1005Metric_Pad0.72x0.64mm_HandSolder
- U701: renamed from U6; value ~ -> ATA6561-GAQW-N; footprint (none) -> Package_SO:SOIC-8-1EP_3.9x4.9mm_P1.27mm_EP2.41x3.3mm
Changed lines of the file:
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@@
       (effects (font (size 1.27 1.27)) (justify left))
     )
-    (property "Footprint" "" (at 183.8452 101.6 0)
+    (property "Footprint" "Capacitor_SMD:C_0402_1005Metric_Pad0.74x0.62mm_HandSolder" (at 183.8452 101.6 0)
       (effects (font (size 1.27 1.27)) hide)
     )
@@
         )
         (path "/5a70b585-4866-4f79-8013-f2242aeded57/af3f9453-a9b7-4a53-9354-21782482a9ca"
-          (reference "C30") (unit 1)
+          (reference "C701") (unit 1)
         )
       )
@@
         )
         (path "/5a70b585-4866-4f79-8013-f2242aeded57/af3f9453-a9b7-4a53-9354-21782482a9ca"
-          (reference "#PWR074") (unit 1)
+          (reference "#PWR0705") (unit 1)
         )
       )
@@
   (symbol (lib_id "ESC:ATA6561") (at 135.89 96.52 0) (unit 1)
     (in_bom yes) (on_board yes) (dnp no) (fields_autoplaced)
-    (property "Reference" "U6" (at 135.89 87.63 0)
-      (effects (font (size 1.27 1.27)))
-    )
-    (property "Value" "~" (at 135.89 96.52 0)
-      (effects (font (size 1.27 1.27)))
-    )
-    (property "Footprint" "" (at 135.89 96.52 0)
+    (property "Reference" "U701" (at 135.89 87.63 0)
+      (effects (font (size 1.27 1.27)))
+    )
+    (property "Value" "ATA6561-GAQW-N" (at 135.89 96.52 0)
+      (effects (font (size 1.27 1.27)))
+    )
+    (property "Footprint" "Package_SO:SOIC-8-1EP_3.9x4.9mm_P1.27mm_EP2.41x3.3mm" (at 135.89 96.52 0)
       (effects (font (size 1.27 1.27)) hide)
     )
@@
       (project "go-kart-esc"
         (path "/5a70b585-4866-4f79-8013-f2242aeded57/af3f9453-a9b7-4a53-9354-21782482a9ca"
-          (reference "U6") (unit 1)
+          (reference "U701") (unit 1)
         )
       )
@@
         (path "/5a70b585-4866-4f79-8013-f2242aeded57/2f2eb473-a6d5-4b09-8c58-ce0c11f580af"
           (reference "#PWR010") (unit 1)
-        )
-        (path "/5a70b585-4866-4f79-8013-f2242aeded57/49a20c67-eeb7-49f1-8210-196c79304ab5"
-          (reference "#PWR054") (unit 1)
         )
         (path "/5a70b585-4866-4f79-8013-f2242aeded57"
@@
         )
         (path "/5a70b585-4866-4f79-8013-f2242aeded57/af3f9453-a9b7-4a53-9354-21782482a9ca"
-          (reference "#PWR072") (unit 1)
+          (reference "#PWR0702") (unit 1)
         )
       )
@@
         (path "/5a70b585-4866-4f79-8013-f2242aeded57/2f2eb473-a6d5-4b09-8c58-ce0c11f580af"
           (reference "#PWR010") (unit 1)
-        )
-        (path "/5a70b585-4866-4f79-8013-f2242aeded57/49a20c67-eeb7-49f1-8210-196c79304ab5"
-          (reference "#PWR054") (unit 1)
         )
         (path "/5a70b585-4866-4f79-8013-f2242aeded57"
@@
         )
         (path "/5a70b585-4866-4f79-8013-f2242aeded57/af3f9453-a9b7-4a53-9354-21782482a9ca"
-          (reference "#PWR075") (unit 1)
+          (reference "#PWR0706") (unit 1)
         )
       )
@@
   (symbol (lib_id "power:+5V") (at 152.4 88.9 0) (unit 1)
     (in_bom yes) (on_board yes) (dnp no) (fields_autoplaced)
-    (property "Reference" "#PWR070" (at 152.4 92.71 0)
+    (property "Reference" "#PWR0703" (at 152.4 92.71 0)
       (effects (font (size 1.27 1.27)) hide)
     )
@@
       (project "go-kart-esc"
         (path "/5a70b585-4866-4f79-8013-f2242aeded57/af3f9453-a9b7-4a53-9354-21782482a9ca"
-          (reference "#PWR070") (unit 1)
+          (reference "#PWR0703") (unit 1)
         )
       )
@@
   (symbol (lib_id "power:+5V") (at 182.88 91.44 0) (unit 1)
     (in_bom yes) (on_board yes) (dnp no) (fields_autoplaced)
-    (property "Reference" "#PWR073" (at 182.88 95.25 0)
+    (property "Reference" "#PWR0704" (at 182.88 95.25 0)
       (effects (font (size 1.27 1.27)) hide)
     )
@@
       (project "go-kart-esc"
         (path "/5a70b585-4866-4f79-8013-f2242aeded57/af3f9453-a9b7-4a53-9354-21782482a9ca"
-          (reference "#PWR073") (unit 1)
+          (reference "#PWR0704") (unit 1)
         )
       )
@@
       (effects (font (size 1.27 1.27)) (justify left))
     )
-    (property "Footprint" "" (at 200.3552 101.6 0)
+    (property "Footprint" "Capacitor_SMD:C_0402_1005Metric_Pad0.74x0.62mm_HandSolder" (at 200.3552 101.6 0)
       (effects (font (size 1.27 1.27)) hide)
     )
@@
         )
         (path "/5a70b585-4866-4f79-8013-f2242aeded57/af3f9453-a9b7-4a53-9354-21782482a9ca"
-          (reference "C29") (unit 1)
+          (reference "C702") (unit 1)
         )
       )
@@
         )
         (path "/5a70b585-4866-4f79-8013-f2242aeded57/af3f9453-a9b7-4a53-9354-21782482a9ca"
-          (reference "#PWR071") (unit 1)
+          (reference "#PWR0701") (unit 1)
         )
       )
@@
       (effects (font (size 1.27 1.27)))
     )
-    (property "Value" "220" (at 161.29 99.06 90)
-      (effects (font (size 1.27 1.27)))
-    )
-    (property "Footprint" "" (at 160.528 99.06 90)
+    (property "Value" "120" (at 161.29 99.06 90)
+      (effects (font (size 1.27 1.27)))
+    )
+    (property "Footprint" "Resistor_SMD:R_0402_1005Metric_Pad0.72x0.64mm_HandSolder" (at 160.528 99.06 90)
       (effects (font (size 1.27 1.27)) hide)
     )
@@
         (path "/5a70b585-4866-4f79-8013-f2242aeded57/2f2eb473-a6d5-4b09-8c58-ce0c11f580af"
           (reference "R4") (unit 1)
-        )
-        (path "/5a70b585-4866-4f79-8013-f2242aeded57/49a20c67-eeb7-49f1-8210-196c79304ab5"
-          (reference "R11") (unit 1)
         )
         (path "/5a70b585-4866-4f79-8013-f2242aeded57"
@@
         )
         (path "/5a70b585-4866-4f79-8013-f2242aeded57/af3f9453-a9b7-4a53-9354-21782482a9ca"
-          (reference "R15") (unit 1)
-        )
-      )
+          (reference "R701") (unit 1)
+        )
+      )

Commit message: Finished PCB
Parts:
- renumbered C3 to C701, C3 to C702, R4 to R701
