File: pcb/go-kart-esc/go-kart-esc.kicad_pcb (KiCad board)
At the start: 2 copper layers, 85 parts, among them J101 VBAT, J102 GND, J103 5V_CONN, J104 CAN_CONN, J105 CAN_CONN, J106 TEMP_CONN_A, J107 ENCODER_CONN_A, J108 ENCODER_CONN_B, J109 TEMP_CONN_B, J110 SWD_CONN, J111 THROTTLE_CONN, J112 BRAKE_CONN, J301 MOTOR_A+, J302 MOTOR_A-, J601 MOTOR_A+, J602 MOTOR_A-, Q301 CSD19533Q5A, Q302 CSD19533Q5A, Q303 CSD19533Q5A, Q304 CSD19533Q5A, Q601 CSD19533Q5A, Q602 CSD19533Q5A, Q603 CSD19533Q5A, Q604 CSD19533Q5A, U201 DRV8701PRGER, U301 INA185A2QDCKRQ1, U401 STM32F042C6Ux, U501 DRV8701PRGER, U601 INA185A2QDCKRQ1, U701 ATA6561-GAQW-N

Commit message: ooga booga
Parts:
- C202, C502: value 1u -> 0.1u; footprint Capacitor_SMD:C_0603_1608Metric_Pad1.08x0.95mm_HandSolder -> Capacitor_SMD:C_0402_1005Metric_Pad0.74x0.62mm_HandSolder
- C601, J301, J302, Q301, Q302, Q303, Q304, Q601, Q602, Q603, Q604, R301, R601, U301, U601: moved to B.Cu
- moved C206 138.2 mm to (52.8, 149.5), turned to 180 degrees
- moved U201 134.7 mm to (59.0, 155.6)
- moved C202 133.4 mm to (54.8, 155.5), turned to -90 degrees
- moved C201 132.7 mm to (55.3, 152.4), turned to -90 degrees
- moved C204 131.5 mm to (56.4, 159.5), turned to 180 degrees
- moved C203 131.0 mm to (59.1, 161.0)
- moved C205 130.5 mm to (52.6, 151.5), turned to 180 degrees
- moved R201 129.3 mm to (63.3, 159.0), turned to 180 degrees
- moved R202 127.9 mm to (63.3, 158.0)
- moved R302 50.0 mm to (19.4, 173.6)
- moved C301 50.0 mm to (22.7, 177.4)
- moved TH301 50.0 mm to (22.5, 179.3)
- moved C304 40.2 mm to (42.1, 132.5)
- moved J302 36.1 mm to (53.5, 185.0), turned to 180 degrees
- moved C302 35.0 mm to (74.1, 133.5)
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Connections:
- C201 pad 1: Net-(C201-Pad1) -> +BATT
- C501 pad 1: Net-(C501-Pad1) -> +BATT
- R301 pad 1: /Power-A/MOTOR_LOW -> GND
- R601 pad 1: /Power-A1/MOTOR_LOW -> GND
- U201 pad 25: (no net) -> GND
- U301 pad 1: /Power-A/C -> /Power-A/VREF
- U301 pad 3: /Power-A/SHUNT+ -> +3V3
- U301 pad 4: /Power-A/SHUNT- -> /Power-A/MOTOR_LOW
- U301 pad 5: /Power-A/VREF -> GND
- U301 pad 6: +3V3 -> /Power-A/C
- U501 pad 25: (no net) -> GND
- U601 pad 1: /Power-A1/C -> /Power-A1/VREF
- U601 pad 3: /Power-A1/SHUNT+ -> +3V3
- U601 pad 4: /Power-A1/SHUNT- -> /Power-A1/MOTOR_LOW
- U601 pad 5: /Power-A1/VREF -> GND
- U601 pad 6: +3V3 -> /Power-A1/C
Routing:
- net (no net): track 0.00 -> 2.12 mm

Commit message: Began Routing
Parts:
- removed C102: 680u, Capacitor_THT:CP_Radial_D16.0mm_P7.50mm
- removed J110: SWD_CONN, Connector_JST:JST_XH_S5B-XH-A_1x05_P2.50mm_Horizontal
- removed R201, R202, R501, R502: 10k, Resistor_SMD:R_0402_1005Metric_Pad0.72x0.64mm_HandSolder
- added C801: 1u, Capacitor_SMD:C_0402_1005Metric_Pad0.74x0.62mm_HandSolder, F.Cu at (93.1, 36.0)
- added C802: 1u, Capacitor_SMD:C_0402_1005Metric_Pad0.74x0.62mm_HandSolder, F.Cu at (93.0, 30.0)
- added U801: MIC5504-3.3YM5, Package_TO_SOT_SMD:SOT-23-5, F.Cu at (92.6, 33.0)
- C201, C203, C204, C501, C503, C504: footprint Capacitor_SMD:C_0603_1608Metric_Pad1.08x0.95mm_HandSolder -> Capacitor_SMD:C_0402_1005Metric_Pad0.74x0.62mm_HandSolder; moved to B.Cu
- C202, C502: value 0.1u -> 0.1u@50V; footprint Capacitor_SMD:C_0402_1005Metric_Pad0.74x0.62mm_HandSolder -> Capacitor_SMD:C_0603_1608Metric_Pad1.08x0.95mm_HandSolder; moved to B.Cu
- C205, C505: value 1u -> 1u@50V; footprint Capacitor_SMD:C_0603_1608Metric_Pad1.08x0.95mm_HandSolder -> Capacitor_SMD:C_0402_1005Metric_Pad0.74x0.62mm_HandSolder; moved to B.Cu
- C206, C506: value 10u -> 10u@50V; footprint Capacitor_SMD:C_0805_2012Metric_Pad1.18x1.45mm_HandSolder -> Capacitor_SMD:CP_Elec_5x5.8
- C303, C603, R302, R305, R602, R605, TH301, TH601, U201, U501: moved to B.Cu
- C408: footprint Capacitor_SMD:C_0603_1608Metric_Pad1.08x0.95mm_HandSolder -> Capacitor_SMD:C_0402_1005Metric_Pad0.74x0.62mm_HandSolder
- C601, J301, J302, Q301, Q302, Q303, Q304, Q601, Q602, Q603, Q604, R301, R601, U301, U601: moved to F.Cu
- J105: value CAN_CONN -> SWD_CONN; footprint Connector_JST:JST_XH_S2B-XH-A_1x02_P2.50mm_Horizontal -> Connector_PinHeader_2.54mm:PinHeader_2x02_P2.54mm_Vertical
- moved C405 164.2 mm to (56.5, 43.3)
- moved C407 158.8 mm to (56.2, 45.8)
- moved U401 154.5 mm to (57.3, 53.7), turned to -90 degrees
- moved C403 153.8 mm to (50.0, 56.3), turned to 90 degrees
- moved C406 153.5 mm to (66.5, 50.9), turned to -90 degrees
- moved C408 152.0 mm to (59.9, 62.5), turned to 180 degrees
- moved C401 151.3 mm to (57.9, 47.0)
- moved C404 148.2 mm to (64.0, 50.9), turned to -90 degrees
- moved C402 142.4 mm to (59.9, 60.2), turned to 180 degrees
- moved R701 141.2 mm to (70.0, 34.0), turned to 180 degrees
- moved C702 134.3 mm to (73.6, 38.6), turned to -90 degrees
- moved U701 134.0 mm to (70.0, 40.5), turned to 90 degrees
- moved C701 131.6 mm to (70.1, 45.0), turned to 180 degrees
- moved J301 119.4 mm to (20.5, 75.0), turned to -90 degrees
- moved C506 118.4 mm to (65.0, 98.5)
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Connections:
- C101 pad 1: Net-(C101-Pad1) -> +BATT
- C402 pad 1: Net-(C402-Pad1) -> +3V3
- C403 pad 1: Net-(C402-Pad1) -> +3V3
- C404 pad 1: Net-(C402-Pad1) -> +3V3
- C405 pad 1: Net-(C402-Pad1) -> +3V3
- C406 pad 1: Net-(C402-Pad1) -> +3V3
- C407 pad 1: Net-(C402-Pad1) -> +3V3
- C408 pad 1: Net-(C402-Pad1) -> +3V3
- J105 pad 1: /CAN/CANL -> /STM32F042/nRESET
- J105 pad 2: /CAN/CANH -> /STM32F042/SWDIO
- J301 pad 1: /DRV8701P-A/SH1 -> /DRV8701P-A/SH2
- J302 pad 1: /DRV8701P-A/SH2 -> /DRV8701P-A/SH1
- J601 pad 1: /DRV8701P-A1/SH1 -> /DRV8701P-A1/SH2
- J602 pad 1: /DRV8701P-A1/SH2 -> /DRV8701P-A1/SH1
- Q301 pad 1: /DRV8701P-A/SH1 -> /DRV8701P-A/SH2
- Q301 pad 2: /DRV8701P-A/SH1 -> /DRV8701P-A/SH2
- Q301 pad 3: /DRV8701P-A/SH1 -> /DRV8701P-A/SH2
- Q301 pad 4: /DRV8701P-A/GH1 -> /DRV8701P-A/GH2
- Q302 pad 4: /DRV8701P-A/GL1 -> /DRV8701P-A/GL2
- Q302 pad 5: /DRV8701P-A/SH1 -> /DRV8701P-A/SH2
- Q303 pad 1: /DRV8701P-A/SH2 -> /DRV8701P-A/SH1
- Q303 pad 2: /DRV8701P-A/SH2 -> /DRV8701P-A/SH1
- Q303 pad 3: /DRV8701P-A/SH2 -> /DRV8701P-A/SH1
- Q303 pad 4: /DRV8701P-A/GH2 -> /DRV8701P-A/GH1
- Q304 pad 4: /DRV8701P-A/GL2 -> /DRV8701P-A/GL1
- Q304 pad 5: /DRV8701P-A/SH2 -> /DRV8701P-A/SH1
- Q601 pad 1: /DRV8701P-A1/SH1 -> /DRV8701P-A1/SH2
- Q601 pad 2: /DRV8701P-A1/SH1 -> /DRV8701P-A1/SH2
- Q601 pad 3: /DRV8701P-A1/SH1 -> /DRV8701P-A1/SH2
- Q601 pad 4: /DRV8701P-A1/GH1 -> /DRV8701P-A1/GH2
- Q602 pad 4: /DRV8701P-A1/GL1 -> /DRV8701P-A1/GL2
- Q602 pad 5: /DRV8701P-A1/SH1 -> /DRV8701P-A1/SH2
- Q603 pad 1: /DRV8701P-A1/SH2 -> /DRV8701P-A1/SH1
- Q603 pad 2: /DRV8701P-A1/SH2 -> /DRV8701P-A1/SH1
- Q603 pad 3: /DRV8701P-A1/SH2 -> /DRV8701P-A1/SH1
- Q603 pad 4: /DRV8701P-A1/GH2 -> /DRV8701P-A1/GH1
- Q604 pad 4: /DRV8701P-A1/GL2 -> /DRV8701P-A1/GL1
- Q604 pad 5: /DRV8701P-A1/SH2 -> /DRV8701P-A1/SH1
- U201 pad 12: /DRV8701P-A/IDRIVE -> GND
- U401 pad 25: /DRV8701P-A1/nFAULT -> /DRV8701P-A/nFAULT
- U401 pad 26: /DRV8701P-A1/nSLEEP -> /DRV8701P-A/nSLEEP
- U401 pad 27: /DRV8701P-A/nFAULT -> /DRV8701P-A1/nFAULT
- U401 pad 28: /DRV8701P-A/nSLEEP -> /DRV8701P-A1/nSLEEP
- U401 pad 29: /DRV8701P-A1/IN1 -> /DRV8701P-A/IN2
- U401 pad 30: /DRV8701P-A1/IN2 -> /DRV8701P-A/IN1
- U401 pad 31: /DRV8701P-A/IN1 -> /DRV8701P-A1/IN2
- U401 pad 32: /DRV8701P-A/IN2 -> /DRV8701P-A1/IN1
- U501 pad 12: /DRV8701P-A1/IDRIVE -> GND
Routing:
- net GND: track 0.00 -> 99.6 mm, vias 0 -> 29
- net +3V3: track 0.00 -> 45.1 mm, vias 0 -> 5
- net /STM32F042/WHEEL_ENCODER_B: track 0.00 -> 44.8 mm, vias 0 -> 1
- net /STM32F042/WHEEL_ENCODER_A: track 0.00 -> 44.3 mm, vias 0 -> 1
- net /DRV8701P-A/GH1: track 0.00 -> 44.1 mm, vias 0 -> 1
- net /DRV8701P-A/SH2: track 0.00 -> 43.4 mm, vias 0 -> 1
- net /DRV8701P-A/GH2: track 0.00 -> 41.5 mm, vias 0 -> 1
- net /DRV8701P-A1/nFAULT: track 0.00 -> 40.7 mm, vias 0 -> 1
- net /DRV8701P-A/SH1: track 0.00 -> 40.1 mm, vias 0 -> 1
- net /DRV8701P-A1/IN2: track 0.00 -> 38.9 mm, vias 0 -> 1
- net /DRV8701P-A1/nSLEEP: track 0.00 -> 38.9 mm, vias 0 -> 1
- net /DRV8701P-A1/IN1: track 0.00 -> 38.6 mm, vias 0 -> 1
- net /DRV8701P-A/GL2: track 0.00 -> 35.1 mm, vias 0 -> 1
- net /DRV8701P-A/IN1: track 0.00 -> 34.9 mm, vias 0 -> 1
- net /DRV8701P-A/IN2: track 0.00 -> 33.5 mm, vias 0 -> 1
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- added copper zone on F.Cu, net +3V3
- added copper zone on In2.Cu, net +3V3
- added copper zone on F.Cu, net +5V
- added copper zone on In2.Cu, net +5V
- added copper zone on F.Cu, net +BATT
- added copper zone on F.Cu, net /DRV8701P-A/SH1
- added copper zone on F.Cu, net /DRV8701P-A/SH2
- added copper zone on F.Cu, net /DRV8701P-A1/SH1
- added copper zone on F.Cu, net /DRV8701P-A1/SH2
- added copper zone on F.Cu, net /Power-A/MOTOR_LOW
- added copper zone on F.Cu, net /Power-A1/MOTOR_LOW
- added copper zone on F.Cu, net GND
- added copper zone on In1.Cu, net GND
Other:
- copper layers 2 -> 4

Commit message: Theory can only take you so far.
Parts:
- added D104: ESD9B5.0ST5G, Diode_SMD:D_SOD-923, F.Cu at (101.0, 56.0)
- added D106: ESD9B5.0ST5G, Diode_SMD:D_SOD-923, F.Cu at (28.5, 55.5)
- added D108: ESD9B5.0ST5G, Diode_SMD:D_SOD-923, F.Cu at (101.5, 41.0)
- added D110: ESD9B5.0ST5G, Diode_SMD:D_SOD-923, F.Cu at (28.5, 40.5)
- added D112: ESD9B5.0ST5G, Diode_SMD:D_SOD-923, F.Cu at (34.4, 28.5)
- added D114: ESD9B5.0ST5G, Diode_SMD:D_SOD-923, F.Cu at (49.5, 28.5)
- added D116: ESD9B5.0ST5G, Diode_SMD:D_SOD-923, F.Cu at (84.9, 57.0)
- added D117: ESD9B5.0ST5G, Diode_SMD:D_SOD-923, F.Cu at (84.0, 64.5)
- added D118: ESD9B5.0ST5G, Diode_SMD:D_SOD-923, F.Cu at (80.5, 64.5)
- added H401: MountingHole, MountingHole:MountingHole_3.2mm_M3, F.Cu at (20.0, 20.0)
- added H402: MountingHole, MountingHole:MountingHole_3.2mm_M3, F.Cu at (110.0, 20.0)
- added H403: MountingHole, MountingHole:MountingHole_3.2mm_M3, F.Cu at (110.0, 110.0)
- added H404: MountingHole, MountingHole:MountingHole_3.2mm_M3, F.Cu at (20.0, 110.0)
- moved R101 18.4 mm to (30.0, 55.6), turned to -90 degrees
- moved R102 11.1 mm to (99.5, 56.1), turned to -90 degrees
- moved C402 1.16 mm to (61.1, 60.5)
- moved C408 1.16 mm to (61.1, 62.8)
- moved J103 0.60 mm to (96.2, 23.4)
- moved J104 0.50 mm to (71.2, 24.9)
- moved J106 0.50 mm to (24.9, 52.5)
- moved J107 0.50 mm to (24.9, 37.5)
- moved J108 0.50 mm to (105.0, 42.5)
- moved J109 0.50 mm to (105.0, 57.5)
- moved J111 0.50 mm to (52.5, 24.9)
- moved J112 0.50 mm to (37.5, 24.9)
Connections:
- C203 pad 1: +3V3 -> Net-(U201-DVDD)
- C204 pad 1: +4V -> Net-(U201-AVDD)
- C503 pad 1: +3V3 -> Net-(U501-DVDD)
- C504 pad 1: +4V -> Net-(U501-AVDD)
- U201 pad 7: +4V -> Net-(U201-AVDD)
- U201 pad 8: +3V3 -> Net-(U201-DVDD)
- U501 pad 7: +4V -> Net-(U501-AVDD)
- U501 pad 8: +3V3 -> Net-(U501-DVDD)
Routing:
- net /Power-A1/TEMP: track 0.00 -> 92.0 mm, vias 0 -> 1
- net /Power-A/TEMP: track 0.00 -> 62.6 mm, vias 0 -> 1
- net /Power-A1/CURR: track 18.0 -> 79.9 mm, vias 0 -> 1
- net /STM32F042/MOTOR_TEMP_B: track 0.00 -> 58.7 mm, vias 0 -> 2
- net /Power-A/CURR: track 8.47 -> 42.6 mm, vias 0 -> 1
- net /STM32F042/BRAKE: track 0.00 -> 33.9 mm
- net /STM32F042/MOTOR_TEMP_A: track 0.00 -> 29.7 mm
- net /STM32F042/THROTTLE: track 0.00 -> 27.4 mm
- net GND: track 99.6 -> 122.4 mm, vias 29 -> 219
- net /STM32F042/WHEEL_ENCODER_A: track 44.3 -> 58.1 mm, vias 1 -> 4
- net /STM32F042/nRESET: track 32.6 -> 42.3 mm
- net +3V3: track 45.1 -> 53.6 mm, vias 5 -> 29
- net /STM32F042/WHEEL_ENCODER_B: track 44.8 -> 51.4 mm, vias 1 -> 2
- net Net-(U501-DVDD): track 0.00 -> 6.17 mm, vias 0 -> 1
- net Net-(U201-DVDD): track 0.00 -> 6.08 mm, vias 0 -> 1
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- added copper zone on B.Cu, net GND
Other:
- board outline added: 100 x 100 mm

Commit message: Finished PCB
Parts:
- added J401: CAN_CONN, Connector_JST:JST_XH_S2B-XH-A_1x02_P2.50mm_Horizontal, F.Cu at (84.2, 24.9)
- TH301, TH601: footprint Resistor_SMD:R_0201_0603Metric_Pad0.64x0.40mm_HandSolder -> Resistor_SMD:R_0402_1005Metric_Pad0.72x0.64mm_HandSolder
Routing:
- net /CAN/CANH: track 13.4 -> 28.3 mm
- net /CAN/CANL: track 14.3 -> 28.9 mm
Other:
- board text added: "3v3"
- board text added: "5V"
- board text added: "A+"
- board text added: "A-"
- board text added: "B+"
- board text added: "B-"
- board text added: "BRAKE"
- board text added: "CAN HIGH"
- board text added: "CAN LOW"
- board text added: "GND"
- board text added: "MOTOR ENCODER A"
- board text added: "MOTOR TEMP A"
- board text added: "MOTOR TMP B"
- board text added: "PA2 - THROTTLE PA3 - BRAKE PA4 - CURRENT A PA5 - TEMP A PA6 - CURRENT B PA7 - TEMP B PB6 - LED GREEN PB7 - LED RED PB3 - WHEEL ENCODER A PA15 - WHEEL ENCODER B PB12 - nFAULT A PB13 - nSLEEP A PB14 - nFAULT B PB15 - nSLEEP B PA8 - A- PA9 - A+ PA10 - B+ PA11 - B-"
- board text added: "SWCLK"
- board text added: "SWDIO"
- board text added: "THROTTLE"
- board text added: "VBAT"
- board text added: "WHEEL ENCODER B"
- board text added: "nRESET"
