File: pcb/go-kart-esc/go-kart-esc.kicad_sch (KiCad schematic)
At the start: 0 parts

Commit message: Poggers
Parts:
- added C9 (x2): 680u, symbol Device:C_Polarized
- added D1: BLUE, symbol Device:LED
- added D2: GREEN, symbol Device:LED
- added D3: RED, symbol Device:LED
- added J10: SWD, symbol Connector_Generic:Conn_01x05
- added J11: TEMP_CONN_A, Connector_JST:JST_PH_S3B-PH-K_1x03_P2.00mm_Horizontal, symbol Connector_Generic:Conn_01x03
- added J12: TEMP_CONN_B, Connector_JST:JST_PH_S3B-PH-K_1x03_P2.00mm_Horizontal, symbol Connector_Generic:Conn_01x03
- added J13: ENCODER_CONN_A, Connector_JST:JST_PH_S3B-PH-K_1x03_P2.00mm_Horizontal, symbol Connector_Generic:Conn_01x03
- added J14: ENCODER_CONN_B, Connector_JST:JST_PH_S3B-PH-K_1x03_P2.00mm_Horizontal, symbol Connector_Generic:Conn_01x03
- added J5: BRAKE_CONN, Connector_JST:JST_PH_S3B-PH-K_1x03_P2.00mm_Horizontal, symbol Connector_Generic:Conn_01x03
- added J6: THROTTLE_CONN, Connector_JST:JST_PH_S3B-PH-K_1x03_P2.00mm_Horizontal, symbol Connector_Generic:Conn_01x03
- added J7, J9: CAN_CONN, symbol Connector_Generic:Conn_01x02
- added J8: 5V_CONN, symbol Connector_Generic:Conn_01x02
- added R4: 10, symbol Device:R
- added R5 (x2): 10k, symbol Device:R
Connections:
- new net: C9.1, C9.1
- new net: D3.1 (K), R4.1
- new net +3V3: D1.2 (A), J10.5 (Pin_5), J11.3 (Pin_3), J12.3 (Pin_3), J13.3 (Pin_3), J14.3 (Pin_3), J5.3 (Pin_3), J6.3 (Pin_3)
- new net +5V: J8.2 (Pin_2)
- new net CAN/CANH: J7.2 (Pin_2), J9.2 (Pin_2)
- new net CAN/CANL: J7.1 (Pin_1), J9.1 (Pin_1)
- new net GND: C9.2, C9.2, D1.1 (K), D2.1 (K), J10.3 (Pin_3), J11.1 (Pin_1), J12.1 (Pin_1), J13.1 (Pin_1), J14.1 (Pin_1), J5.1 (Pin_1), J6.1 (Pin_1), J8.1 (Pin_1), R4.2, R5.2, R5.2
- new net STM32F042/BRAKE: J5.2 (Pin_2)
- new net STM32F042/LED_GREEN: D2.2 (A)
- new net STM32F042/LED_RED: D3.2 (A)
- new net STM32F042/MOTOR_TEMP_A: J11.2 (Pin_2), R5.1
- new net STM32F042/MOTOR_TEMP_B: J12.2 (Pin_2), R5.1
- new net STM32F042/SWCLK: J10.4 (Pin_4)
- new net STM32F042/SWDIO: J10.2 (Pin_2)
- new net STM32F042/THROTTLE: J6.2 (Pin_2)
- new net STM32F042/WHEEL_ENCODER_A: J13.2 (Pin_2)
- new net STM32F042/WHEEL_ENCODER_B: J14.2 (Pin_2)
- new net STM32F042/nRESET: J10.1 (Pin_1)
Other:
- added sheet CAN (can.kicad_sch)
- added sheet DRV8701P-A1 (DRV8701P-A.kicad_sch)
- added sheet Power-A1 (power-a.kicad_sch)
- added sheet STM32F042 (STM32F042.kicad_sch)
- sheet Power-A ports: added CURR, TEMP; removed none

Commit message: ooga booga
Parts:
- added J1: VBAT, ESC:Motor_Solder_Pad, symbol Connector_Generic:Conn_01x01
- added J3: GND, ESC:Motor_Solder_Pad, symbol Connector_Generic:Conn_01x01
- C9: footprint (none) -> Capacitor_THT:CP_Radial_D16.0mm_P7.50mm
- D101: renamed from D1; footprint (none) -> LED_SMD:LED_0603_1608Metric_Pad1.05x0.95mm_HandSolder
- D102: renamed from D2; footprint (none) -> LED_SMD:LED_0603_1608Metric_Pad1.05x0.95mm_HandSolder
- D103: renamed from D3; footprint (none) -> LED_SMD:LED_0603_1608Metric_Pad1.05x0.95mm_HandSolder
- J103: renamed from J8; footprint (none) -> Connector_JST:JST_XH_S2B-XH-A-1_1x02_P2.50mm_Horizontal
- J104: renamed from J7; footprint (none) -> Connector_JST:JST_XH_S2B-XH-A_1x02_P2.50mm_Horizontal
- J105: renamed from J9; footprint (none) -> Connector_JST:JST_XH_S2B-XH-A_1x02_P2.50mm_Horizontal
- J106: renamed from J11; footprint Connector_JST:JST_PH_S3B-PH-K_1x03_P2.00mm_Horizontal -> Connector_JST:JST_XH_S3B-XH-A_1x03_P2.50mm_Horizontal
- J107: renamed from J13; footprint Connector_JST:JST_PH_S3B-PH-K_1x03_P2.00mm_Horizontal -> Connector_JST:JST_XH_S3B-XH-A_1x03_P2.50mm_Horizontal
- J108: renamed from J14; footprint Connector_JST:JST_PH_S3B-PH-K_1x03_P2.00mm_Horizontal -> Connector_JST:JST_XH_S3B-XH-A_1x03_P2.50mm_Horizontal
- J109: renamed from J12; footprint Connector_JST:JST_PH_S3B-PH-K_1x03_P2.00mm_Horizontal -> Connector_JST:JST_XH_S3B-XH-A_1x03_P2.50mm_Horizontal
- J110: renamed from J10; value SWD -> SWD_CONN; footprint (none) -> Connector_JST:JST_XH_S5B-XH-A_1x05_P2.50mm_Horizontal
- J111: renamed from J6; footprint Connector_JST:JST_PH_S3B-PH-K_1x03_P2.00mm_Horizontal -> Connector_JST:JST_XH_S3B-XH-A_1x03_P2.50mm_Horizontal
- J112: renamed from J5; footprint Connector_JST:JST_PH_S3B-PH-K_1x03_P2.00mm_Horizontal -> Connector_JST:JST_XH_S3B-XH-A_1x03_P2.50mm_Horizontal
- R4: footprint (none) -> Resistor_SMD:R_0603_1608Metric_Pad0.98x0.95mm_HandSolder
- R5: footprint (none) -> Resistor_SMD:R_0402_1005Metric_Pad0.72x0.64mm_HandSolder
Connections:
- net GND: now also J3.1 (Pin_1)
- new net +BATT: J1.1 (Pin_1)
Other:
- moved on the sheet: D101

Commit message: Began Routing
Parts:
- removed C9: 680u, Capacitor_THT:CP_Radial_D16.0mm_P7.50mm, symbol Device:C_Polarized
- removed J105: CAN_CONN, Connector_JST:JST_XH_S2B-XH-A_1x02_P2.50mm_Horizontal, symbol Connector_Generic:Conn_01x02
- removed J110: SWD_CONN, Connector_JST:JST_XH_S5B-XH-A_1x05_P2.50mm_Horizontal, symbol Connector_Generic:Conn_01x05
- added J105: SWD_CONN, Connector_PinHeader_2.54mm:PinHeader_2x02_P2.54mm_Vertical, symbol Connector_Generic:Conn_01x04
Connections:
- net +BATT: now also C9.1
- net GND: now also J105.3 (Pin_3)
- net STM32F042/SWCLK: now also J105.4 (Pin_4)
- net STM32F042/SWDIO: now also J105.2 (Pin_2)
- net STM32F042/nRESET: now also J105.1 (Pin_1)
Other:
- added sheet 3v3 LDO (3v3_LDO.kicad_sch)

Commit message: Theory can only take you so far.
Parts:
- added D104, D106, D108, D110, D112, D114, D116, D117, D118: ESD9B5.0ST5G, Diode_SMD:D_SOD-923, symbol Diode:ESD9B5.0ST5G
- added H401, H402, H403, H404: MountingHole, MountingHole:MountingHole_3.2mm_M3, symbol Mechanical:MountingHole
Connections:
- net GND: now also D104.1 (A1), D106.1 (A1), D108.1 (A1), D110.1 (A1), D112.1 (A1), D114.1 (A1), D116.1 (A1), D117.1 (A1), D118.1 (A1)
- net STM32F042/BRAKE: now also D112.2 (A2)
- net STM32F042/MOTOR_TEMP_A: now also D106.2 (A2)
- net STM32F042/MOTOR_TEMP_B: now also D104.2 (A2)
- net STM32F042/SWCLK: now also D118.2 (A2)
- net STM32F042/SWDIO: now also D117.2 (A2)
- net STM32F042/THROTTLE: now also D114.2 (A2)
- net STM32F042/WHEEL_ENCODER_A: now also D110.2 (A2)
- net STM32F042/WHEEL_ENCODER_B: now also D108.2 (A2)
- net STM32F042/nRESET: now also D116.2 (A2)
Other:
- moved on the sheet: J107, J108, J109

Commit message: Finished PCB
Parts:
- added J401: CAN_CONN, Connector_JST:JST_XH_S2B-XH-A_1x02_P2.50mm_Horizontal, symbol Connector_Generic:Conn_01x02
- renumbered C9 to C101, J1 to J101, J3 to J102, R5 to R101, R5 to R102, R4 to R103
Connections:
- net CAN/CANH: now also J401.2 (Pin_2)
- net CAN/CANL: now also J401.1 (Pin_1)
